File: Revised Keyboard/Revised Version Of 60%/Revised Version Of 60%.kicad_pcb (KiCad board)
At the start: 2 copper layers, 247.7 x 83.3 mm, 104 parts, among them J1 AVR-ISP-6, SW1 SW_Push, U1 AT90USB1286-A, U2 PRTR5V0U2X, Y1 Crystal_GND24_Small

Commit message: Update
General Update of files
Parts:
- moved J1 31.8 mm to (514.1, 147.4)
- moved C3 20.4 mm to (533.5, 141.5), turned to 90 degrees
- moved R3 16.3 mm to (541.8, 156.7)
- moved C4 1.09 mm to (535.3, 138.2), turned to 90 degrees
Connections:
- U1 pad 1: unconnected-(U1-Pad1) -> GND
- U1 pad 44: unconnected-(U1-Pad44) -> GND
- U1 pad 45: unconnected-(U1-Pad45) -> SCK
- U1 pad 46: unconnected-(U1-Pad46) -> MOSI
- U1 pad 47: unconnected-(U1-Pad47) -> MISO
- U1 pad 49: MISO -> unconnected-(U1-Pad49)
- U1 pad 50: MOSI -> unconnected-(U1-Pad50)
- U1 pad 51: SCK -> unconnected-(U1-Pad51)
Routing:
- net GND: track 120.8 -> 216.7 mm, vias 4 -> 7
- net +5V: track 97.6 -> 134.8 mm, vias 6 -> 8
- net Net-(R3-Pad1): track 0.00 -> 2.46 mm
- net MISO: track 0.00 -> 0.80 mm
- net MOSI: track 0.00 -> 0.76 mm
- net SCK: track 0.00 -> 0.73 mm

Commit message: Keyboard Update
Changed to a smaller microcontroller
Parts:
- removed the MX_SPACEBAR1 at (569.9, 146.1)
- removed R3, R4: 10k, Resistor_SMD:R_0805_2012Metric_Pad1.20x1.40mm_HandSolder
- added C8: 1u, Capacitor_SMD:C_0805_2012Metric, F.Cu at (666.8, -41.4)
- added R1: 10k, Resistor_SMD:R_0805_2012Metric_Pad1.20x1.40mm_HandSolder, F.Cu at (707.5, -81.8)
- C1, C2, C3: value 0.1uF -> 0.1u; moved to F.Cu
- C4: value 10uF -> 0.1u; moved to F.Cu
- C5: value 22pF -> 10u; moved to F.Cu
- C6: value 22pF -> 22p; moved to F.Cu
- C7: value 1uF -> 22p; moved to F.Cu
- F1, J1, R5, R6, R7, R8, SW1, U2, USB1, Y1: moved to F.Cu
- MX_RSHIFT1: moved to B.Cu
- MX_SPACEBAR1: renamed from R1; value 22 -> MX-NoLED; footprint Resistor_SMD:R_0805_2012Metric_Pad1.20x1.40mm_HandSolder -> MX_Alps_Hybrid:MX-6.5U-NoLED; moved to F.Cu
- R2: value 22 -> 10k; moved to F.Cu
- U1: value AT90USB1286-A -> ATmega32U4-A; footprint Package_QFP:TQFP-64_14x14mm_P0.8mm -> Package_QFP:TQFP-44_10x10mm_P0.8mm; moved to F.Cu
- moved R8 271.7 mm to (713.2, -88.1), turned to 0 degrees
- moved R2 234.4 mm to (666.9, -44.4), turned to 0 degrees
- moved R5 230.5 mm to (707.5, -84.8)
- moved R6 183.6 mm to (672.7, -47.7), turned to 0 degrees
- moved F1 171.6 mm to (606.9, -67.1), turned to 0 degrees
- moved U2 156.5 mm to (652.5, -27.0), turned to 0 degrees
- moved SW1 145.1 mm to (500.5, 36.0), turned to 0 degrees
- moved C4 142.0 mm to (608.7, 16.5), turned to 0 degrees
- moved C2 138.0 mm to (608.7, 13.5), turned to 0 degrees
- moved Y1 118.6 mm to (514.8, 35.7), turned to 0 degrees
- moved C3 118.3 mm to (588.7, 36.7), turned to 0 degrees
- moved C5 117.9 mm to (508.7, 42.6), turned to 0 degrees
- moved C6 114.1 mm to (588.7, 33.7), turned to 0 degrees
- moved C1 111.5 mm to (503.9, 42.6), turned to 0 degrees
- moved J1 110.8 mm to (508.4, 36.8), turned to 0 degrees
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Connections:
- C1 pad 1: +5V -> GND
- C1 pad 2: GND -> +5V
- C2 pad 1: +5V -> GND
- C2 pad 2: GND -> +5V
- C5 pad 2: Net-(C5-Pad2) -> +5V
- C6 pad 1: GND -> XTAL1
- C6 pad 2: Net-(C6-Pad2) -> GND
- C7 pad 1: Net-(C7-Pad1) -> XTAL2
- J1 pad 2: VCC -> +5V
- J1 pad 5: Net-(J1-Pad5) -> RESET
- MX_SPACEBAR1 pad 1: Net-(R1-Pad1) -> Net-(MX_H1-Pad1)
- MX_SPACEBAR1 pad 2: D+ -> Net-(D_SPACEBAR1-Pad2)
- R2 pad 1: Net-(R2-Pad1) -> GND
- R2 pad 2: D- -> Net-(R2-Pad2)
- SW1 pad 1: Net-(J1-Pad5) -> GND
- SW1 pad 2: GND -> RESET
- U1 pad 1: GND -> unconnected-(U1-Pad1)
- U1 pad 10: unconnected-(U1-Pad10) -> MOSI
- U1 pad 11: unconnected-(U1-Pad11) -> SCK
- U1 pad 13: unconnected-(U1-Pad13) -> RESET
- U1 pad 14: unconnected-(U1-Pad14) -> +5V
- U1 pad 15: unconnected-(U1-Pad15) -> GND
- U1 pad 16: unconnected-(U1-Pad16) -> XTAL2
- U1 pad 17: unconnected-(U1-Pad17) -> XTAL1
- U1 pad 2: unconnected-(U1-Pad2) -> +5V
- U1 pad 20: Net-(J1-Pad5) -> unconnected-(U1-Pad20)
- U1 pad 21: +5V -> unconnected-(U1-Pad21)
- U1 pad 22: GND -> unconnected-(U1-Pad22)
- U1 pad 23: Net-(C6-Pad2) -> GND
- U1 pad 24: Net-(C5-Pad2) -> +5V
- U1 pad 29: unconnected-(U1-Pad29) -> Column 1
- U1 pad 3: +5V -> D-
- U1 pad 33: unconnected-(U1-Pad33) -> Net-(R2-Pad2)
- U1 pad 34: unconnected-(U1-Pad34) -> +5V
- U1 pad 35: unconnected-(U1-Pad35) -> GND
- U1 pad 4: D- -> D+
- U1 pad 43: Net-(R3-Pad1) -> GND
- U1 pad 44: GND -> +5V
- U1 pad 5: D+ -> GND
- U1 pad 6: GND -> Net-(C8-Pad1)
- U1 pad 7: Net-(C7-Pad1) -> unconnected-(U1-Pad7)
- U1 pad 8: +5V -> unconnected-(U1-Pad8)
- U1 pad 9: unconnected-(U1-Pad9) -> MISO
- Y1 pad 1: Net-(C5-Pad2) -> XTAL1
- Y1 pad 3: Net-(C6-Pad2) -> XTAL2
Routing:
- net GND: track 216.7 -> 0.00 mm, vias 7 -> 0
- net Net-(D_BACKSPACE1-Pad1): track 201.3 -> 0.00 mm
- net Net-(D_(1-Pad1): track 196.1 -> 0.00 mm
- net Net-(D_?1-Pad1): track 187.3 -> 0.00 mm
- net Net-(D_ALT1-Pad1): track 147.2 -> 0.00 mm
- net +5V: track 134.8 -> 0.00 mm, vias 8 -> 0
- net Net-(MX_?1-Pad1): track 82.3 -> 0.00 mm
- net Net-(MX_)1-Pad1): track 73.3 -> 0.00 mm
- net Net-(MX_A1-Pad1): track 70.2 -> 0.00 mm
- net Net-(MX_H1-Pad1): track 69.7 -> 0.00 mm
- net DP: track 68.6 -> 0.00 mm
- net Net-(MX_ALT1-Pad1): track 68.2 -> 0.00 mm
- net DN: track 66.7 -> 0.00 mm
- net Net-(MX_CTRL1-Pad1): track 66.3 -> 0.00 mm
- net Net-(MX_J1-Pad1): track 48.2 -> 0.00 mm
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- removed copper zone on B.Cu, net GND
- removed copper zone on F.Cu, net GND
Other:
- board size 247.7 x 83.3 mm -> 243 x 76.3 mm

Commit message: Keyboard Nearly finished
All components wired up on the PCB
Parts:
- removed C2: 0.1u, Capacitor_SMD:C_0805_2012Metric_Pad1.18x1.45mm_HandSolder
- removed J1: AVR-ISP-6, random-keyboard-parts:Reset_Pretty-Mask
- C1, C3, C4, C5, C6, C7, C8, F1, R1, R2, R5, R6, R7, R8, SW1, U1, U2, USB1, Y1: moved to B.Cu
- moved R8 310.5 mm to (571.0, 187.8), turned to 90 degrees
- moved R1 291.3 mm to (614.8, 194.3), turned to 180 degrees
- moved R2 274.1 mm to (560.1, 208.0)
- moved R5 271.5 mm to (558.2, 142.0)
- moved C8 250.7 mm to (573.7, 191.4), turned to 90 degrees
- moved F1 226.6 mm to (551.7, 152.7), turned to -90 degrees
- moved R6 224.3 mm to (553.0, 142.0), turned to 180 degrees
- moved U2 201.4 mm to (555.9, 149.7), turned to 180 degrees
- moved SW1 197.6 mm to (611.8, 199.4), turned to 180 degrees
- moved C4 184.9 mm to (557.8, 194.3)
- moved C1 179.8 mm to (574.3, 208.0), turned to -90 degrees
- moved Y1 178.4 mm to (579.6, 201.9), turned to 90 degrees
- moved C7 176.0 mm to (584.3, 200.5)
- moved C3 171.1 mm to (557.5, 205.0), turned to -90 degrees
- moved C6 169.8 mm to (584.3, 203.5)
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Connections:
- D_(1 pad 1: Net-(D_(1-Pad1) -> Row 3
- D_)1 pad 1: Net-(D_(1-Pad1) -> Row 3
- D_?1 pad 1: Net-(D_?1-Pad1) -> Row 2
- D_A1 pad 1: Net-(D_?1-Pad1) -> Row 2
- D_ALT1 pad 1: Net-(D_ALT1-Pad1) -> Row 4
- D_B1 pad 1: Net-(D_(1-Pad1) -> Row 3
- D_BACKSPACE1 pad 1: Net-(D_BACKSPACE1-Pad1) -> Row 1
- D_C1 pad 1: Net-(D_(1-Pad1) -> Row 3
- D_CAPS1 pad 1: Net-(D_ALT1-Pad1) -> Row 4
- D_CTRL1 pad 1: Net-(D_ALT1-Pad1) -> Row 4
- D_D1 pad 1: Net-(D_?1-Pad1) -> Row 2
- D_E1 pad 1: Net-(D_BACKSPACE1-Pad1) -> Row 1
- D_ESC1 pad 1: Net-(D_BACKSPACE1-Pad1) -> Row 1
- D_Enter1 pad 1: Net-(D_?1-Pad1) -> Row 2
- D_F1 pad 1: Net-(D_?1-Pad1) -> Row 2
- D_FN1 pad 1: Net-(D_ALT1-Pad1) -> Row 4
- D_G1 pad 1: Net-(D_?1-Pad1) -> Row 2
- D_H1 pad 1: Net-(D_?1-Pad1) -> Row 2
- D_I1 pad 1: Net-(D_BACKSPACE1-Pad1) -> Row 1
- D_J1 pad 1: Net-(D_?1-Pad1) -> Row 2
- D_K1 pad 1: Net-(D_?1-Pad1) -> Row 2
- D_L1 pad 1: Net-(D_?1-Pad1) -> Row 2
- D_M1 pad 1: Net-(D_(1-Pad1) -> Row 3
- D_N1 pad 1: Net-(D_(1-Pad1) -> Row 3
- D_O1 pad 1: Net-(D_BACKSPACE1-Pad1) -> Row 1
- D_P1 pad 1: Net-(D_BACKSPACE1-Pad1) -> Row 1
- D_Q1 pad 1: Net-(D_BACKSPACE1-Pad1) -> Row 1
- D_R1 pad 1: Net-(D_BACKSPACE1-Pad1) -> Row 1
- D_RSHIFT1 pad 1: Net-(D_(1-Pad1) -> Row 3
- D_S1 pad 1: Net-(D_?1-Pad1) -> Row 2
- D_SHIFT1 pad 1: Net-(D_(1-Pad1) -> Row 3
- D_SPACEBAR1 pad 1: Net-(D_ALT1-Pad1) -> Row 4
- D_SUPER1 pad 1: Net-(D_ALT1-Pad1) -> Row 4
- D_T1 pad 1: Net-(D_BACKSPACE1-Pad1) -> Row 1
- D_TAB1 pad 1: Net-(D_?1-Pad1) -> Row 2
- D_U1 pad 1: Net-(D_BACKSPACE1-Pad1) -> Row 1
- D_V1 pad 1: Net-(D_(1-Pad1) -> Row 3
- D_W1 pad 1: Net-(D_BACKSPACE1-Pad1) -> Row 1
- D_X1 pad 1: Net-(D_(1-Pad1) -> Row 3
- D_Y1 pad 1: Net-(D_BACKSPACE1-Pad1) -> Row 1
- D_Z1 pad 1: Net-(D_(1-Pad1) -> Row 3
- MX_(1 pad 1: Net-(MX_(1-Pad1) -> Column 9
- MX_)1 pad 1: Net-(MX_)1-Pad1) -> Column 10
- MX_?1 pad 1: Net-(MX_?1-Pad1) -> Column 11
- MX_A1 pad 1: Net-(MX_A1-Pad1) -> Column 2
- MX_ALT1 pad 1: Net-(MX_ALT1-Pad1) -> Column 3
- MX_B1 pad 1: Net-(MX_B1-Pad1) -> Column 6
- MX_BACKSPACE1 pad 1: Net-(MX_BACKSPACE1-Pad1) -> Column 12
- MX_C1 pad 1: Net-(MX_C1-Pad1) -> Column 4
- MX_CAPS1 pad 1: Net-(MX_?1-Pad1) -> Column 11
- MX_CTRL1 pad 1: Net-(MX_CTRL1-Pad1) -> Column 1
- MX_D1 pad 1: Net-(MX_C1-Pad1) -> Column 4
- MX_E1 pad 1: Net-(MX_C1-Pad1) -> Column 4
- MX_ENTER1 pad 1: Net-(MX_BACKSPACE1-Pad1) -> Column 12
- MX_ESC1 pad 1: Net-(MX_CTRL1-Pad1) -> Column 1
- MX_F1 pad 1: Net-(MX_F1-Pad1) -> Column 5
- MX_FN1 pad 1: Net-(MX_)1-Pad1) -> Column 10
- MX_G1 pad 1: Net-(MX_B1-Pad1) -> Column 6
- MX_H1 pad 1: Net-(MX_H1-Pad1) -> Column 7
- MX_I1 pad 1: Net-(MX_(1-Pad1) -> Column 9
- MX_J1 pad 1: Net-(MX_J1-Pad1) -> Column 8
- MX_K1 pad 1: Net-(MX_(1-Pad1) -> Column 9
- MX_L1 pad 1: Net-(MX_)1-Pad1) -> Column 10
- MX_M1 pad 1: Net-(MX_J1-Pad1) -> Column 8
- MX_N1 pad 1: Net-(MX_H1-Pad1) -> Column 7
- MX_O1 pad 1: Net-(MX_)1-Pad1) -> Column 10
- MX_P1 pad 1: Net-(MX_?1-Pad1) -> Column 11
- MX_Q1 pad 1: Net-(MX_A1-Pad1) -> Column 2
- MX_R1 pad 1: Net-(MX_F1-Pad1) -> Column 5
- MX_RSHIFT1 pad 1: Net-(MX_?1-Pad1) -> Column 11
- MX_S1 pad 1: Net-(MX_ALT1-Pad1) -> Column 3
- MX_SHIFT1 pad 1: Net-(MX_CTRL1-Pad1) -> Column 1
- MX_SPACEBAR1 pad 1: Net-(MX_H1-Pad1) -> Column 7
- MX_SUPER1 pad 1: Net-(MX_A1-Pad1) -> Column 2
- MX_T1 pad 1: Net-(MX_B1-Pad1) -> Column 6
- MX_TAB1 pad 1: Net-(MX_CTRL1-Pad1) -> Column 1
- MX_U1 pad 1: Net-(MX_J1-Pad1) -> Column 8
- MX_V1 pad 1: Net-(MX_F1-Pad1) -> Column 5
- MX_W1 pad 1: Net-(MX_ALT1-Pad1) -> Column 3
- MX_X1 pad 1: Net-(MX_ALT1-Pad1) -> Column 3
- MX_Y1 pad 1: Net-(MX_H1-Pad1) -> Column 7
- MX_Z1 pad 1: Net-(MX_A1-Pad1) -> Column 2
- U1 pad 10: MOSI -> Column 6
- U1 pad 11: SCK -> Column 7
- U1 pad 12: unconnected-(U1-Pad12) -> Column 8
- U1 pad 19: unconnected-(U1-Pad19) -> Column 9
- U1 pad 20: unconnected-(U1-Pad20) -> Column 10
- U1 pad 21: unconnected-(U1-Pad21) -> Column 11
- U1 pad 22: unconnected-(U1-Pad22) -> Column 12
- U1 pad 29: Column 1 -> Row 4
- U1 pad 30: unconnected-(U1-Pad30) -> Row 3
- U1 pad 31: unconnected-(U1-Pad31) -> Row 2
- U1 pad 32: unconnected-(U1-Pad32) -> Row 1
- U1 pad 37: unconnected-(U1-Pad37) -> Column 1
- U1 pad 38: unconnected-(U1-Pad38) -> Column 2
- U1 pad 39: unconnected-(U1-Pad39) -> Column 3
- U1 pad 40: unconnected-(U1-Pad40) -> Column 4
- U1 pad 41: unconnected-(U1-Pad41) -> Column 5
- U1 pad 7: unconnected-(U1-Pad7) -> +5V
- U1 pad 9: MISO -> unconnected-(U1-Pad9)
Routing:
- net Row 1: track 0.00 -> 324.5 mm, vias 0 -> 4
- net Row 2: track 0.00 -> 302.7 mm, vias 0 -> 4
- net Row 3: track 0.00 -> 297.9 mm, vias 0 -> 2
- net GND: track 0.00 -> 235.4 mm, vias 0 -> 9
- net Row 4: track 0.00 -> 228.5 mm
- net Column 12: track 0.00 -> 209.9 mm, vias 0 -> 1
- net Column 11: track 0.00 -> 202.9 mm, vias 0 -> 1
- net +5V: track 0.00 -> 182.9 mm, vias 0 -> 7
- net Column 10: track 0.00 -> 172.1 mm, vias 0 -> 1
- net Column 1: track 0.00 -> 170.9 mm, vias 0 -> 1
- net Column 2: track 0.00 -> 152.1 mm, vias 0 -> 1
- net Column 9: track 0.00 -> 136.3 mm, vias 0 -> 1
- net Column 3: track 0.00 -> 126.2 mm, vias 0 -> 1
- net Column 8: track 0.00 -> 104.0 mm, vias 0 -> 1
- net Column 7: track 0.00 -> 96.8 mm, vias 0 -> 1
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- added copper zone on B.Cu, net GND
- added copper zone on F.Cu, net GND
Other:
- board size 243 x 76.3 mm -> 243 x 82.6 mm
